File: uC.sch (KiCad schematic (older format))
At the start: 0 parts

Commit message: k20 symbol added
created parts library and added k20 schematic to it.
uc hierarchical page now located on main page of schematic.
Parts:
- added U?: MK20DX256VLH7, MODULE, symbol MK20DX256VLH7
Other:
- note removed: "0"
- note removed: "2015-03-11"
- note removed: "Pixel - block diagram"
Changed lines of the file:
@@
 LIBS:contrib
 LIBS:valves
+LIBS:pixel_pcb_r0
 LIBS:pixel_pcb_r0-cache
 EELAYER 25 0
 EELAYER END
-$Descr D 34000 22000
+$Descr C 22000 17000
 encoding utf-8
-Sheet 1 2
+Sheet 2 2
 Title ""
 Date ""
@@
 Comment4 ""
 $EndDescr
-Text Notes 30450 21350 0    60   ~ 0
-2015-03-11
-Text Notes 29650 21250 0    60   ~ 0
-Pixel - block diagram
-Text Notes 32900 21350 0    60   ~ 0
-0
-$Sheet
-S 20500 4750 2600 2600
-U 551787C3
-F0 "uC" 60
-F1 "uC.sch" 60
-$EndSheet
+$Comp
+L MK20DX256VLH7 U?
+U 1 1 5517B259
+P 10950 8500
+F 0 "U?" H 10950 8400 50  0000 C CNN
+F 1 "MK20DX256VLH7" H 10950 9550 50  0000 C CNN
+F 2 "MODULE" H 10950 9450 50  0001 C CNN
+F 3 "DOCUMENTATION" H 10950 9450 50  0001 C CNN
+	1    10950 8500
+	1    0    0    -1
+$EndComp
 $EndSCHEMATC
